File: KICAD/iplanter.kicad_pcb (KiCad board)
At the start: 2 copper layers, 64 x 71.5 mm, 5 parts, among them J1 Moisture Sensor, J2 Display, J3 DHT11, J4 Barrel_Jack_MountingPin, U2 WEMOS_D1_mini

Commit message: Add files via upload
Parts:
- moved U2 28.2 mm to (93.2, 87.3), turned to 180 degrees
Routing:
- net Net-(U2-5V): track 46.2 -> 77.6 mm
- net /AOUT: track 57.3 -> 29.3 mm
- net /SDA: track 70.0 -> 50.8 mm
- net Net-(J3-Pin_2): track 32.2 -> 13.1 mm
- net /SCL: track 57.0 -> 48.1 mm
- added copper zone on F.Cu, net /GND
- removed copper zone on B.Cu, net /GND
